File: RTR-CANSystem-board/RTR-CANSystem-board.kicad_sch (KiCad schematic)
At the start: 19 parts, among them J1 MicroB, J2 USB_A, J3 USB_A, J4 Conn_01x07_Socket, J5 Conn_01x07_Socket, SW1 RESET, SW2 BOOT, U2 NJM72223, U3 ESP32-C3-WROOM-02

Commit message: Yちゃんに焼きそば一口もらった
Parts:
- removed J5: Conn_01x07_Socket, symbol 01.RTR-CANSystem-board_library:Conn_01x07_Socket
- added J5: Conn_01x08_Socket, 01.RTR-CANSystem-board_library:PinHeader_1x08_P2.54mm_Vertical, symbol 01.RTR-CANSystem-board_library:Conn_01x08_Socket
- C1, C2, C3, C4, C5, C6: footprint (none) -> 01.RTR-CANSystem-board_library:C_0603_1608Metric_Pad1.08x0.95mm_HandSolder
- J1: footprint ZX62-B-5PA_33_:HRS_ZX62-B-5PA_33_ -> 01.RTR-CANSystem-board_library:HRS_ZX62-B-5PA_33_
- J2: footprint (none) -> 01.RTR-CANSystem-board_library:USB_A_CNCTech_1001-011-01101_Horizontal
- J3: footprint (none) -> 01.RTR-CANSystem-board_library:usb-PCB
- J4: footprint (none) -> 01.RTR-CANSystem-board_library:PinHeader_1x07_P2.54mm_Vertical
- R1: footprint (none) -> 01.RTR-CANSystem-board_library:R_Axial_DIN0204_L3.6mm_D1.6mm_P7.62mm_Horizontal
- R2, R3: value R_Small -> 10k; footprint (none) -> 01.RTR-CANSystem-board_library:R_0805_2012Metric
- SW1, SW2: footprint (none) -> 01.RTR-CANSystem-board_library:SW_Push_1P1T_NO_CK_KSC7xxJ
- U1: footprint (none) -> 01.RTR-CANSystem-board_library:DIP-8_W7.62mm
- U2: footprint digikey-footprints:TO-220-3 -> 01.RTR-CANSystem-board_library:TO-252-2
- U3: footprint PCM_Espressif:ESP32-C3-WROOM-02 -> 01.RTR-CANSystem-board_library:ESP32-C3-WROOM-02
Connections:
- net 3.3V: now also J5.6 (Pin_6)
- net 5V: now also J5.8 (Pin_8)
- net CANH: now also J5.5 (Pin_5)
- net CANL: now also U1.6 (CANL), J5.4 (Pin_4); no longer U1.4 (RXD)
- net GND: now also J5.7 (Pin_7)
- net GPIO10: now also J5.1 (Pin_1)
- net GPIO20: now also J5.2 (Pin_2)
- net GPIO21: now also J5.3 (Pin_3)
- no-connect marks 2 -> 1
Other:
- moved on the sheet: J4
